File: Firmware/pcb/login-controller/login-controller.kicad_pcb (KiCad board)
At the start: 2 copper layers, 100 x 84 mm, 19 parts, among them J1 Conn_01x02, J2 Conn_01x02, J4 Conn_ARM_JTAG_SWD_10, SW1 SW_DIP_x08, U1 ESP32-DEVKITC-32D, U2 pn532_breakout, U3 Micro_SD_Card_module, U4 L7805

Commit message: Firmware: DIP Switch added
Connections:
- R2 pad 1: +3V3 -> GND
- R3 pad 1: +3V3 -> GND
- R4 pad 1: +3V3 -> GND
- R5 pad 1: +3V3 -> GND
- R6 pad 1: +3V3 -> GND
- R7 pad 1: +3V3 -> GND
- R8 pad 1: +3V3 -> GND
- R9 pad 1: +3V3 -> GND
- SW1 pad 10: GND -> +3V3
- SW1 pad 11: GND -> +3V3
- SW1 pad 12: GND -> +3V3
- SW1 pad 13: GND -> +3V3
- SW1 pad 14: GND -> +3V3
- SW1 pad 15: GND -> +3V3
- SW1 pad 16: GND -> +3V3
- SW1 pad 9: GND -> +3V3
Routing:
- net +3V3: track 160.0 -> 124.9 mm, vias 2 -> 1
- net GND: track 0.00 -> 20.7 mm, vias 0 -> 1
