File: Firmware/pcb/login-controller/login-controller.kicad_sch (KiCad schematic)
At the start: 19 parts, among them J1 Conn_01x02, J2 Conn_01x02, J4 Conn_ARM_JTAG_SWD_10, SW1 SW_DIP_x08, U1 ESP32-DEVKITC-32D, U2 pn532_breakout, U3 Micro_SD_Card_module, U4 L7805

Commit message: Firmware: DIP Switch added
Connections:
- net +3V3: now also SW1.10, SW1.11, SW1.12, SW1.13, SW1.14, SW1.15, SW1.16, SW1.9; no longer R2.1, R3.1, R4.1, R5.1, R6.1, R7.1, R8.1, R9.1
- net GND: now also R2.1, R3.1, R4.1, R5.1, R6.1, R7.1, R8.1, R9.1; no longer SW1.10, SW1.11, SW1.12, SW1.13, SW1.14, SW1.15, SW1.16, SW1.9
Changed lines of the file:
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@@
   (junction (at 105.41 179.07) (diameter 0) (color 0 0 0 0)
   )
+  (junction (at 105.41 189.23) (diameter 0) (color 0 0 0 0)
+  )
   (junction (at 83.82 137.16) (diameter 0) (color 0 0 0 0)
   )
@@
   (junction (at 105.41 181.61) (diameter 0) (color 0 0 0 0)
   )
+  (junction (at 148.59 171.45) (diameter 0) (color 0 0 0 0)
+  )
   (junction (at 58.42 137.16) (diameter 0) (color 0 0 0 0)
   )
   (junction (at 71.12 151.13) (diameter 0) (color 0 0 0 0)
   )
-  (junction (at 148.59 189.23) (diameter 0) (color 0 0 0 0)
-  )
   (junction (at 148.59 181.61) (diameter 0) (color 0 0 0 0)
   )
@@
   )
   (junction (at 148.59 179.07) (diameter 0) (color 0 0 0 0)
-  )
-  (junction (at 105.41 171.45) (diameter 0) (color 0 0 0 0)
   )
   (junction (at 148.59 176.53) (diameter 0) (color 0 0 0 0)
@@
   )
   (wire (pts (xy 148.59 176.53) (xy 148.59 179.07))
-    (stroke (width 0) (type default) (color 0 0 0 0))
-  )
-  (wire (pts (xy 105.41 167.64) (xy 105.41 171.45))
     (stroke (width 0) (type default) (color 0 0 0 0))
   )
@@
     (pin "6")
   )
-  (symbol (lib_id "power:+3V3") (at 105.41 167.64 0) (unit 1)
-    (in_bom yes) (on_board yes) (fields_autoplaced)
-    (property "Reference" "#PWR0117" (id 0) (at 105.41 171.45 0)
-      (effects (font (size 1.27 1.27)) hide)
-    )
-    (property "Value" "+3V3" (id 1) (at 105.41 162.56 0))
-    (property "Footprint" "" (id 2) (at 105.41 167.64 0)
-      (effects (font (size 1.27 1.27)) hide)
-    )
-    (property "Datasheet" "" (id 3) (at 105.41 167.64 0)
+  (symbol (lib_id "power:+3V3") (at 148.59 171.45 0) (unit 1)
+    (in_bom yes) (on_board yes) (fields_autoplaced)
+    (property "Reference" "#PWR0117" (id 0) (at 148.59 175.26 0)
+      (effects (font (size 1.27 1.27)) hide)
+    )
+    (property "Value" "+3V3" (id 1) (at 148.59 166.37 0))
+    (property "Footprint" "" (id 2) (at 148.59 171.45 0)
+      (effects (font (size 1.27 1.27)) hide)
+    )
+    (property "Datasheet" "" (id 3) (at 148.59 171.45 0)
       (effects (font (size 1.27 1.27)) hide)
     )
@@
     (pin "1")
   )
-  (symbol (lib_id "power:GND") (at 148.59 189.23 0) (unit 1)
-    (in_bom yes) (on_board yes) (fields_autoplaced)
-    (property "Reference" "#PWR0116" (id 0) (at 148.59 195.58 0)
-      (effects (font (size 1.27 1.27)) hide)
-    )
-    (property "Value" "GND" (id 1) (at 148.59 194.31 0))
-    (property "Footprint" "" (id 2) (at 148.59 189.23 0)
-      (effects (font (size 1.27 1.27)) hide)
-    )
-    (property "Datasheet" "" (id 3) (at 148.59 189.23 0)
-      (effects (font (size 1.27 1.27)) hide)
-    )
+  (symbol (lib_id "power:GND") (at 105.41 189.23 0) (unit 1)
+    (in_bom yes) (on_board yes) (fields_autoplaced)
+    (property "Reference" "#PWR0116" (id 0) (at 105.41 195.58 0)
+      (effects (font (size 1.27 1.27)) hide)
+    )
+    (property "Value" "GND" (id 1) (at 105.41 194.31 0))
+    (property "Footprint" "" (id 2) (at 105.41 189.23 0)
+      (effects (font (size 1.27 1.27)) hide)
+    )
+    (property "Datasheet" "" (id 3) (at 105.41 189.23 0)
+      (effects (font (size 1.27 1.27)) hide)
+    )
